Commit message: working in rviz and gazebo(turning still not corrected)

File: install/simple_car/share/simple_car/urdf/simple_car.urdf (robot description, URDF)
Before this commit: robot simple_car, 5 links, 4 joints
Links:
- added link base_link
Joints:
- added joint base_to_chassis: type fixed, parent base_link, child chassis, origin xyz=0 0 0.1 rpy=0 0 0
- joint left_front_joint: origin xyz=0.15 0.2 -0.05 rpy=1.5708 0 0 -> xyz=0.15 0.175 -0.1 rpy=1.5708 0 0
- joint left_rear_joint: origin xyz=-0.15 0.2 -0.05 rpy=1.5708 0 0 -> xyz=-0.15 0.175 -0.1 rpy=1.5708 0 0
- joint right_front_joint: origin xyz=0.15 -0.2 -0.05 rpy=1.5708 0 0 -> xyz=0.15 -0.175 -0.1 rpy=1.5708 0 0
- joint right_rear_joint: origin xyz=-0.15 -0.2 -0.05 rpy=1.5708 0 0 -> xyz=-0.15 -0.175 -0.1 rpy=1.5708 0 0
